Commit message: Organizing unit tests. Typo fixes.

File: tests/data/error_incorrect_joint_child_link_name.urdf (robot description, URDF)
Before this commit: robot error_check, 2 links, 1 joints
Joints:
- joint JointA: child link2 -> link_dummy; parent BaseLink_dummy -> BaseLink

File: tests/data/error_incorrect_joint_parent_link_name.urdf (robot description, URDF)
Before this commit: robot error_check, 2 links, 0 joints
Joints:
- added joint JointA: type fixed, parent BaseLink_dummy, child link2
