Commit message: Convert link and joints: Fixing errors, added unit tests

File: tests/data/simple_fixed_planar_joints.urdf (robot description, URDF)
Before this commit: robot simple_fixed_planar_joints, 3 links, 2 joints
Links:
- removed link Arm:1
- removed link Arm:2
- added link link1; visual box size=0.2 0.2 0.2
- added link planar_negative_x; visual box size=0.1 1.0 1.0
- added link planar_negative_y; visual box size=1.0 0.1 1.0
- added link planar_negative_z; visual box size=1.0 1.0 0.1
- added link planar_tilt; visual box size=0.5 0.5 0.1
- added link planar_tilt_axis_len_0; visual box size=0.5 0.5 0.1
- added link planar_x; visual box size=0.1 1.0 1.0
- added link planar_y; visual box size=1.0 0.1 1.0
- added link planar_z; visual box size=1.0 1.0 0.1
Joints:
- removed joint joint_arm:1
- added joint joint_planar_axis_negaive_x: type planar, parent link1, child planar_negative_x, origin xyz=-2 0 0 rpy=0 0 0, axis -1 0 0
- added joint joint_planar_axis_negative_y: type planar, parent link1, child planar_negative_y, origin xyz=0 2 0 rpy=0 0 0, axis 0 -1 0
- added joint joint_planar_axis_negative_z: type planar, parent link1, child planar_negative_z, origin xyz=0 0 0.7 rpy=0 0 0, axis 0 0 -1
- added joint joint_planar_axis_tilt: type planar, parent link1, child planar_tilt, origin xyz=1 0 0 rpy=0 0 0, axis 0.2 0.3 1
- added joint joint_planar_axis_tilt_axis_len_0: type planar, parent link1, child planar_tilt_axis_len_0, origin xyz=1 0 0.5 rpy=0 0 0, axis 0 0 0
- added joint joint_planar_axis_x: type planar, parent link1, child planar_x, origin xyz=-1 0 0 rpy=0 0 0, axis 1 0 0
- added joint joint_planar_axis_y: type planar, parent link1, child planar_y, origin xyz=0 1 0 rpy=0 0 0, axis 0 1 0
- added joint joint_planar_axis_z: type planar, parent link1, child planar_z, origin xyz=0 0 0.35 rpy=0 0 0, axis 0 0 1
- joint joint_root: child Arm:1 -> link1

Commit message: Convert link and joints: Added unit tests for planar joints

File: tests/data/simple_fixed_planar_joints.urdf (robot description, URDF)
Before this commit: robot simple_fixed_planar_joints, 10 links, 9 joints
Joints:
- removed joint joint_planar_axis_negaive_x
- added joint joint_planar_axis_negative_x: type planar, parent link1, child planar_negative_x, origin xyz=-2 0 0 rpy=0 0 0, axis -1 0 0
