Commit message: Adjust parser. Some errors have been moved to warnings.

File: tests/data/warning_missing_collision_geometry.urdf (robot description, URDF)
Before this commit: robot missing_visual_geometry, 1 links, 0 joints
Links:
- link BaseLink: geometry visual box size=1 1 1

File: tests/data/warning_missing_visual_geometry.urdf (robot description, URDF)
Before this commit: robot missing_collision_geometry, 1 links, 0 joints
Links:
- link BaseLink: geometry 
