Commit message: Updated unit tests and urdf files. Converter adjustments.

File: tests/data/fixed_continuous_joints.urdf (robot description, URDF)
Before this commit: robot simple_fixed_floating_joints, 3 links, 2 joints
Links:
- removed link Arm:1
- removed link Arm:2
- added link Arm_1; visual box size=1.0 0.2 0.2
- added link Arm_2; visual box size=1.0 0.2 0.2
Joints:
- removed joint joint_arm:1
- added joint joint_arm_1: type continuous, parent Arm_1, child Arm_2, origin xyz=1.1 0 0.0 rpy=0 0 0, axis 1 0 0
- joint joint_root: child Arm:1 -> Arm_1

File: tests/data/fixed_floating_joints.urdf (robot description, URDF)
Before this commit: robot simple_fixed_continuous_joints, 3 links, 2 joints
Links:
- removed link Arm:1
- removed link Arm:2
- added link Arm_1; visual box size=1.0 0.2 0.2
- added link Arm_2; visual box size=1.0 0.2 0.2
Joints:
- removed joint joint_arm:1
- added joint joint_arm_1: type floating, parent Arm_1, child Arm_2, origin xyz=1.1 0 0.0 rpy=0 0 0
- joint joint_root: child Arm:1 -> Arm_1

File: tests/data/meshes.urdf (robot description, URDF)
Before this commit: robot simple_meshes, 4 links, 3 joints
Joints:
- joint joint_stl_obj: origin xyz=0 0 0 rpy=0 0 0 -> xyz=1 0 0 rpy=0 0 0

File: tests/data/prismatic_joints.urdf (robot description, URDF)
Before this commit: robot simple_revolute_joints, 5 links, 4 joints
Links:
- removed link Arm:1
- removed link Arm:2
- removed link Arm:3
- removed link Arm:4
- added link Arm_1; visual box size=1.0 0.2 0.2
- added link Arm_2; visual box size=1.0 0.2 0.2
- added link Arm_3; visual box size=1.0 0.2 0.2
- added link Arm_4; visual box size=1.0 0.2 0.2
- added link Arm_5; visual box size=1.0 0.2 0.2
Joints:
- joint joint_arm_1: axis 0 1 0 -> 1 0 0; child Arm:2 -> Arm_2; limit upper=0.3 -> upper=0.5 effort=0 velocity=0.01; parent Arm:1 -> Arm_1; type revolute -> prismatic
- joint joint_arm_2: axis 0 1 0 -> 1 0 0; child Arm:3 -> Arm_3; limit lower=-0.3 -> lower=-0.2 effort=0 velocity=0.01; parent Arm:2 -> Arm_2; type revolute -> prismatic
- joint joint_arm_3: axis 0 1 0 -> 1 0 0; child Arm:4 -> Arm_4; limit lower=-0.3 upper=0.5 -> lower=0 upper=0.5 effort=0 velocity=0.01; parent Arm:3 -> Arm_3; type revolute -> prismatic
- joint joint_root: axis 0 1 0 -> 1 0 0; child Arm:1 -> Arm_1; type revolute -> prismatic

File: tests/data/revolute_joints.urdf (robot description, URDF)
Before this commit: robot simple_prismatic_joints, 6 links, 4 joints
Links:
- removed link Arm:1
- removed link Arm:2
- removed link Arm:3
- removed link Arm:4
- removed link Arm:5
- added link Arm_1; visual box size=1.0 0.2 0.2
- added link Arm_2; visual box size=1.0 0.2 0.2
- added link Arm_3; visual box size=1.0 0.2 0.2
- added link Arm_4; visual box size=1.0 0.2 0.2
Joints:
- joint joint_arm_1: axis 1 0 0 -> 0 1 0; child Arm:2 -> Arm_2; limit upper=0.5 effort=0 velocity=0.01 -> upper=0.3; parent Arm:1 -> Arm_1; type prismatic -> revolute
- joint joint_arm_2: axis 1 0 0 -> 0 1 0; child Arm:3 -> Arm_3; limit lower=-0.2 effort=0 velocity=0.01 -> lower=-0.3; parent Arm:2 -> Arm_2; type prismatic -> revolute
- joint joint_arm_3: axis 1 0 0 -> 0 1 0; child Arm:4 -> Arm_4; limit lower=0 upper=0.5 effort=0 velocity=0.01 -> lower=-0.3 upper=0.5; parent Arm:3 -> Arm_3; type prismatic -> revolute
- joint joint_root: axis 1 0 0 -> 0 1 0; child Arm:1 -> Arm_1; type prismatic -> revolute

File: tests/data/simple-primitives.urdf (robot description, URDF)
Before this commit: robot simple-primitives, 3 links, 2 joints
Links:
- removed link link:sphere
- added link link_sphere; visual sphere radius=0.5
Joints:
- joint joint_cylinder_sphere: child link:sphere -> link_sphere
