Commit message: Address review comments on links with no mass source.
- Warn by default when a rigid body has no mass source, and fail only with strict
- Use one rule for an empty link and a visual-only link: a collision or a positive-mass inertial on the link or a descendant
- Keep a joint to the world inside the articulation by applying ArticulationRootAPI to the non-body root
- Classify each link once in LinkHierarchy as a rigid body, a ghost, or a rigid body with no mass source
- Restore movable fixtures that had inertial added only so conversion would not fail

File: tests/data/fixed_continuous_joints.urdf (robot description, URDF)
Before this commit: robot fixed_continuous_joints, 3 links, 2 joints
Links:
- link Arm_2: mass 1 -> None

File: tests/data/fixed_floating_joints.urdf (robot description, URDF)
Before this commit: robot fixed_floating_joints, 3 links, 2 joints
Links:
- link Arm_2: mass 1 -> None

File: tests/data/fixed_planar_joints.urdf (robot description, URDF)
Before this commit: robot fixed_planar_joints, 10 links, 8 joints
Links:
- link planar_negative_x: mass 1 -> None
- link planar_negative_y: mass 1 -> None
- link planar_negative_z: mass 1 -> None
- link planar_tilt: mass 1 -> None
- link planar_x: mass 1 -> None
- link planar_y: mass 1 -> None
- link planar_z: mass 1 -> None

File: tests/data/link_skip_ghost_link_with_mimic.urdf (robot description, URDF)
Before this commit: robot link_skip_ghost_link_with_mimic, 4 links, 3 joints
Links:
- link linkB: mass 1 -> None

File: tests/data/mimic_joint.urdf (robot description, URDF)
Before this commit: robot mimic_joint, 6 links, 5 joints
Links:
- link linkA: mass 1 -> None
- link linkB: mass 1 -> None
- link linkC: mass 1 -> None
- link linkD: mass 1 -> None

File: tests/data/prismatic_joints.urdf (robot description, URDF)
Before this commit: robot prismatic_joints, 6 links, 4 joints
Links:
- link Arm_1: mass 1 -> None
- link Arm_2: mass 1 -> None
- link Arm_3: mass 1 -> None
- link Arm_4: mass 1 -> None

File: tests/data/revolute_joints.urdf (robot description, URDF)
Before this commit: robot revolute_joints, 5 links, 4 joints
Links:
- link Arm_1: mass 1 -> None
- link Arm_2: mass 1 -> None
- link Arm_3: mass 1 -> None
- link Arm_4: mass 1 -> None
