Commit message: Updated unit tests and urdf files. Converter adjustments.

File: tests/data/fixed_planar_joints.urdf (robot description, URDF)
Before this commit: robot fixed_planar_joints, 10 links, 9 joints
Joints:
- removed joint joint_planar_axis_tilt_axis_len_0

File: tests/data/revolute_joints.urdf (robot description, URDF)
Before this commit: robot revolute_joints, 5 links, 4 joints
Joints:
- joint joint_arm_1: origin xyz=1.1 0 0.0 rpy=0 0 0 -> xyz=1.1 0 0.0 rpy=0 0 0.3
- joint joint_arm_2: origin xyz=1.1 0 0.0 rpy=0 0 0 -> xyz=1.1 0 0.1 rpy=0 -0.3 -0.15
- joint joint_arm_3: origin xyz=1.1 0 0.0 rpy=0 0 0 -> xyz=1.1 0.1 0.0 rpy=-0.15 0 0
