Commit message: Custom attributes: urdf:limit:effort, urdf:limit:velocity

File: tests/data/prismatic_joints.urdf (robot description, URDF)
Before this commit: robot prismatic_joints, 6 links, 4 joints
Joints:
- joint joint_arm_1: limit upper=0.5 effort=0 velocity=0.01 -> upper=0.5 effort=0.01
- joint joint_arm_2: limit lower=-0.2 effort=0 velocity=0.01 -> lower=-0.2 effort=0.02 velocity=0.01
- joint joint_arm_3: limit lower=0 upper=0.5 effort=0 velocity=0.01 -> lower=0 upper=0.5 effort=0.03 velocity=0.01

File: tests/data/revolute_joints.urdf (robot description, URDF)
Before this commit: robot revolute_joints, 5 links, 4 joints
Joints:
- joint joint_arm_3: limit lower=-0.3 upper=0.5 -> lower=-0.3 upper=0.5 effort=0.01 velocity=0.02
