Commit message: obj materials: If the texture file does not exist, the path is not passed to USD.
obj materials: Added specular, specular texture, alpha texture

File: tests/data/material_mesh_color.urdf (robot description, URDF)
Before this commit: robot material_mesh_color, 2 links, 1 joints
Links:
- added link link_obj_specular_workflow; visual mesh filename=assets/box_specular_workflow.obj scale=0.5 0.5 0.5
Joints:
- added joint joint_box_obj_specular_workflow: type fixed, parent link_obj, child link_obj_specular_workflow, origin xyz=1 0 0 rpy=0 0 0

File: tests/data/material_mesh_texture.urdf (robot description, URDF)
Before this commit: robot material_mesh_texture, 2 links, 1 joints
Links:
- added link link_obj_opacity; visual mesh filename=assets/box_with_texture_opacity.obj scale=0.5 0.5 0.5
- added link link_obj_specular_workflow_with_texture; visual mesh filename=assets/box_specular_workflow_with_texture.obj scale=0.5 0.5 0.5
Joints:
- added joint joint_box_obj_opacity: type fixed, parent link_obj, child link_obj_opacity, origin xyz=1 0 0 rpy=0 0 0
- added joint joint_box_obj_specular_workflow_with_texture: type fixed, parent link_obj_opacity, child link_obj_specular_workflow_with_texture, origin xyz=1 0 0 rpy=0 0 0
