Commit message: Convert obj to usd

File: tests/data/meshes.urdf (robot description, URDF)
Before this commit: robot meshes, 4 links, 3 joints
Links:
- added link link_mesh_multi_objs; collision mesh filename=assets/two_boxes.obj scale=0.8 0.8 0.8; visual mesh filename=assets/two_boxes.obj scale=0.8 0.8 0.8
- link link_mesh_obj: geometry collision mesh filename=assets/box.obj scale=0.8 0.8 0.8; visual mesh filename=assets/box.obj scale=0.8 0.8 0.8
Joints:
- added joint joint_obj_multi_objs: type fixed, parent link_mesh_stl, child link_mesh_multi_objs, origin xyz=-1 0 0 rpy=0 0 0

File: tests/data/test_displayname.urdf (robot description, URDF)
Before this commit: robot test_displayname, 2 links, 1 joints
Links:
- added link link-mesh_obj; visual mesh filename=assets/name_test.obj scale=0.5 0.5 0.5
Joints:
- added joint mesh_obj: type fixed, parent link-box2, child link-mesh_obj, origin xyz=1 0 0 rpy=0 0 0

Commit message: rebase: Convert dae to usd

File: tests/data/meshes.urdf (robot description, URDF)
Before this commit: robot meshes, 5 links, 4 joints
Links:
- added link link_mesh_dae_unit_cm; visual mesh filename=assets/box_unit_cm.dae scale=0.8 0.8 0.8
- added link link_two_meshes_dae; visual mesh filename=assets/two_meshes.dae scale=0.6 0.6 0.6
- added link link_two_meshes_triangle_dae; visual mesh filename=assets/two_meshes_triangle.dae scale=0.6 0.6 0.6
- link link_mesh_dae: geometry collision mesh filename=assets/box.dae scale=0.8 0.8 0.8; visual mesh filename=assets/box.dae scale=0.8 0.8 0.8
Joints:
- removed joint joint_dae_dxf
- removed joint joint_obj_dae
- added joint joint_dae_multiple: type fixed, parent link_mesh_dae, child link_two_meshes_dae, origin xyz=3.0 0 0 rpy=0 0 1.570796
- added joint joint_dae_multiple_triangle: type fixed, parent link_two_meshes_dae, child link_two_meshes_triangle_dae, origin xyz=0 -2.0 0 rpy=0 0 3.1415926
- added joint joint_dae_unit_cm: type fixed, parent link_mesh_dae, child link_mesh_dae_unit_cm, origin xyz=1.5 0 0 rpy=0 0 0
- added joint joint_stl_dae: type fixed, parent link_mesh_stl, child link_mesh_dae, origin xyz=2.0 0 0 rpy=0 0 0
- added joint joint_stl_dxf: type fixed, parent link_mesh_stl, child link_mesh_dxf, origin xyz=-1 0 0 rpy=0 0 0

File: tests/data/test_displayname.urdf (robot description, URDF)
Before this commit: robot test_displayname, 3 links, 2 joints
Links:
- added link link-mesh_dae; visual mesh filename=assets/name_test.dae scale=0.5 0.5 0.5
Joints:
- added joint mesh_dae: type fixed, parent link-box2, child link-mesh_dae, origin xyz=0 1 0 rpy=0 0 0

Commit message: dae: Removed up-axis.
Adjustments when using multiple primitives.

File: tests/data/meshes.urdf (robot description, URDF)
Before this commit: robot meshes, 8 links, 7 joints
Links:
- added link link_box_two_materials_dae; visual mesh filename=assets/box_two_materials.dae
Joints:
- added joint joint_dae_two_materials: type fixed, parent link_two_meshes_triangle_dae, child link_box_two_materials_dae, origin xyz=0 0 2.0 rpy=0 0 0

Commit message: Convert DAE to USD (#36)

File: tests/data/meshes.urdf (robot description, URDF)
Before this commit: robot meshes, 5 links, 4 joints
Links:
- added link link_box_two_materials_dae; visual mesh filename=assets/box_two_materials.dae
- added link link_mesh_dae_unit_cm; visual mesh filename=assets/box_unit_cm.dae scale=0.8 0.8 0.8
- added link link_two_meshes_dae; visual mesh filename=assets/two_meshes.dae scale=0.6 0.6 0.6
- added link link_two_meshes_triangle_dae; visual mesh filename=assets/two_meshes_triangle.dae scale=0.6 0.6 0.6
- link link_mesh_dae: geometry collision mesh filename=assets/box.dae scale=0.8 0.8 0.8; visual mesh filename=assets/box.dae scale=0.8 0.8 0.8
Joints:
- removed joint joint_dae_dxf
- removed joint joint_obj_dae
- added joint joint_dae_multiple: type fixed, parent link_mesh_dae, child link_two_meshes_dae, origin xyz=3.0 0 0 rpy=0 0 1.570796
- added joint joint_dae_multiple_triangle: type fixed, parent link_two_meshes_dae, child link_two_meshes_triangle_dae, origin xyz=0 -2.0 0 rpy=0 0 3.1415926
- added joint joint_dae_two_materials: type fixed, parent link_two_meshes_triangle_dae, child link_box_two_materials_dae, origin xyz=0 0 2.0 rpy=0 0 0
- added joint joint_dae_unit_cm: type fixed, parent link_mesh_dae, child link_mesh_dae_unit_cm, origin xyz=1.5 0 0 rpy=0 0 0
- added joint joint_stl_dae: type fixed, parent link_mesh_stl, child link_mesh_dae, origin xyz=2.0 0 0 rpy=0 0 0
- added joint joint_stl_dxf: type fixed, parent link_mesh_stl, child link_mesh_dxf, origin xyz=-1 0 0 rpy=0 0 0

File: tests/data/test_displayname.urdf (robot description, URDF)
Before this commit: robot test_displayname, 3 links, 2 joints
Links:
- added link link-mesh_dae; visual mesh filename=assets/name_test.dae scale=0.5 0.5 0.5
Joints:
- added joint mesh_dae: type fixed, parent link-box2, child link-mesh_dae, origin xyz=0 1 0 rpy=0 0 0
