Commit message: dae materials: Adjust opaque_mode

File: tests/data/dae_materials.urdf (robot description, URDF)
Before this commit: robot dae_materials, 2 links, 1 joints
Links:
- added link link_transparent; visual mesh filename=assets/box_transparent_material.dae
Joints:
- added joint joint_link_transparent: type fixed, parent link2, child link_transparent, origin xyz=2 0 0 rpy=0 0 0
