Commit message: Skipped double replacement during material overwriting

File: tests/data/material_mesh_override.urdf (robot description, URDF)
Before this commit: robot material_mesh_override, 2 links, 1 joints
Links:
- added link link_dae; visual mesh filename=assets/box.dae scale=0.5 0.5 0.5
Joints:
- added joint joint_obj_dae: type fixed, parent link_obj, child link_dae, origin xyz=1 0 0 rpy=0 0 0
