Commit message: dae: Changed to use material ID for material identification within one dae.

File: tests/data/test_displayname.urdf (robot description, URDF)
Before this commit: robot test_displayname, 4 links, 3 joints
Links:
- added link link-box_two_materials_same_names; visual mesh filename=assets/box_two_materials_same_names.dae scale=0.5 0.5 0.5
Joints:
- added joint box_two_materials_same_names: type fixed, parent link-box2, child link-box_two_materials_same_names, origin xyz=0 3 0 rpy=0 0 0
