Commit message: Fixed a bug where all the body0 components of joints would become root prims when a Ghost Link was present

File: tests/data/link_first_ghost_link_fixed.urdf (robot description, URDF)
Before this commit: robot link_first_ghost_link_fixed, 2 links, 1 joints
Links:
- added link link_box; collision box size=0.5 0.5 0.5; visual box size=0.5 0.5 0.5
Joints:
- added joint joint_box: type fixed, parent link1, child link_box, origin xyz=0 0 0.8 rpy=0 0 0

File: tests/data/link_first_ghost_link_floating.urdf (robot description, URDF)
Before this commit: robot link_first_ghost_link_floating, 2 links, 1 joints
Links:
- added link link_box; collision box size=0.5 0.5 0.5; visual box size=0.5 0.5 0.5
Joints:
- added joint joint_box: type fixed, parent link1, child link_box, origin xyz=0 0 0.8 rpy=0 0 0
