Commit message: Ghost link: Changed the implementation of Ghost Link processing.

File: tests/data/link_skip_ghost_link.urdf (robot description, URDF)
Before this commit: robot link_skip_ghost_link, 3 links, 2 joints
Links:
- removed link link_box
Joints:
- removed joint joint_box

File: tests/data/link_skip_ghost_link_chain_branch.urdf (robot description, URDF)
Before this commit: robot link_skip_ghost_link_chain, 5 links, 4 joints
Links:
- added link ghost_link_4
- added link ghost_link_5
Joints:
- added joint joint4: type fixed, parent ghost_link_2, child ghost_link_4, origin xyz=0.5 0 0.1 rpy=0 0 0
- added joint joint5: type fixed, parent ghost_link_4, child ghost_link_5, origin xyz=0 0 0.1 rpy=0 0 0

File: tests/data/link_skip_ghost_link_chain_end.urdf (robot description, URDF)
Before this commit: robot link_skip_ghost_link_chain, 5 links, 4 joints
Links:
- removed link link_box
Joints:
- removed joint joint_box
