Commit message: Bug fix for URDF materials with no material name

File: tests/data/verifying_elements.urdf (robot description, URDF)
Before this commit: robot verifying_elements, 3 links, 2 joints
Links:
- added link link4; visual cylinder length=1 radius=0.5
Joints:
- added joint JointC: type fixed, parent link3, child link4, origin xyz=0 0 2 rpy=0 0 0

Commit message: Enhance error checking for Mimic Joint

File: tests/data/verifying_elements.urdf (robot description, URDF)
Before this commit: robot verifying_elements, 4 links, 3 joints
Joints:
- joint JointA: type fixed -> revolute

Commit message: Enhance error checking for Mimic Joint

File: tests/data/verifying_elements.urdf (robot description, URDF)
Before this commit: robot verifying_elements, 4 links, 3 joints
Joints:
- joint JointA: type revolute -> fixed
