Commit message: Ghost link: Updated unit test

File: tests/data/link_ghost_link_inertial_zero.urdf (robot description, URDF)
Before this commit: robot link_ghost_link_inertial_zero, 3 links, 2 joints
Links:
- added link boxLink; collision box size=0.5 0.5 0.5; visual box size=0.5 0.5 0.5
- link ghost_link_no_inertia: mass None -> 0.0
Joints:
- added joint joint1: type fixed, parent BaseLink, child boxLink, origin xyz=0 0 0.1 rpy=0 0 0
- joint joint_no_inertia: parent BaseLink -> boxLink
- joint joint_zero_mass: parent BaseLink -> boxLink
