Commit message: Fix principal axes orientation extracted from the URDF inertia tensor
np.linalg.eigh returns the principal axes as the columns of the
eigenvector matrix, but extract_inertia filled Gf.Matrix3d with it
row-major. Gf matrices use the row-vector convention, so the quaternion
extracted from that matrix was the conjugate (inverse) of the intended
rotation: for any link with non-zero products of inertia, the authored
physics:principalAxes did not reconstruct the URDF inertia tensor via
R * diag * R^T (correct eigenvalues, wrong orientation).

Fill the matrix with the transpose so the extracted rotation maps the
principal frame to the link frame.

Update the expected quaternions in testPhysicsInertia to the corrected
convention (link_box6 is a 180 degree rotation and is unchanged), add a
link_box7 fixture with a non-zero inertial origin rpy combined with all
products of inertia to cover the rpy composition in apply_inertial, and
add a reconstruction assertion that verifies
R(principalAxes) @ diag(diagonalInertia) @ R^T equals the URDF inertia
tensor for every link, independent of Gf conventions.

File: tests/data/inertia.urdf (robot description, URDF)
Before this commit: robot inertia, 6 links, 5 joints
Links:
- added link link_box7, mass 0.8; visual box size=0.5 0.5 1.0
Joints:
- added joint joint_box6_box7: type fixed, parent link_box6, child link_box7, origin xyz=0 0 1.2
