Commit message: Author newton:mimicCoef0 in degrees for angular followers
URDF authors <mimic offset> in the follower joint's position units,
radians for revolute and continuous. NewtonMimicAPI documents coef0 in
degrees, so angular followers were authored 180/pi too small. Prismatic
followers were already correct.

The fixture used offset="0.0", which cannot distinguish a missing
conversion from a correct one -- set_schema_attribute skips values
matching the schema default, so the test only asserted the attribute was
unauthored. It now uses a non-zero angular offset and adds a prismatic
mimic pair, so both the conversion and its absence are pinned.

Closes #133. Newton's importer has the matching read-side fix; landing
this without it makes round trips wrong by 180/pi.

Co-Authored-By: Claude Opus 5 (1M context) <noreply@anthropic.com>

File: tests/data/mimic_joint.urdf (robot description, URDF)
Before this commit: robot mimic_joint, 4 links, 3 joints
Links:
- added link linkC; visual box size=0.5 0.2 0.2
- added link linkD; visual box size=0.5 0.2 0.2
Joints:
- added joint jointC: type prismatic, parent linkA, child linkC, origin xyz=0 0 0 rpy=0 0 0, axis 0 1 0, limit lower=-0.7 upper=0.5
- added joint jointD: type prismatic, parent linkB, child linkD, origin xyz=0 0 0 rpy=0 0 0, axis 0 1 0, limit lower=-0.7 upper=0.5, mimic joint=jointC multiplier=2.0 offset=0.25
- joint jointB: mimic joint=jointA multiplier=2.0 offset=0.0 -> joint=jointA multiplier=2.0 offset=0.5
