Commit message: Added pair-degenerate large-inertia link and conversion E2E coverage

File: tests/data/inertia_large_degenerate.urdf (robot description, URDF)
Before this commit: robot inertia_large_degenerate, 1 links, 0 joints
Links:
- added link link_pair_degenerate_large, mass 1.0; visual box size=0.1 0.1 0.1
Joints:
- added joint joint_isotropic_to_pair: type fixed, parent link_isotropic_large, child link_pair_degenerate_large, origin xyz=0 0 0.2 rpy=0 0 0
