Commit message: Added unit test. If the joint does not have an 'origin' specified.

File: tests/data/dummy_inertia_offset.urdf (robot description, URDF)
Before this commit: robot dummy_inertia_offset, 2 links, 1 joints
Links:
- added link side; collision box size=0.2 0.2 0.2
- added link side_inertia, mass 4
Joints:
- added joint side_inertia_joint: type fixed, parent side, child side_inertia
- added joint side_joint: type revolute, parent base, child side, origin xyz=0.2 0 0 rpy=0 0 0, axis 0 0 1
