Commit message: Stop authoring a visual-only link as a rigid body without mass
A fixed-joint child is treated as a ghost link. A movable joint fails conversion.

File: tests/data/change_joint_order.urdf (robot description, URDF)
Before this commit: robot change_joint_order, 3 links, 2 joints
Links:
- link link_box2: mass None -> 1
- link link_box3: mass None -> 1

File: tests/data/fixed_continuous_joints.urdf (robot description, URDF)
Before this commit: robot fixed_continuous_joints, 3 links, 2 joints
Links:
- link Arm_1: mass None -> 1
- link Arm_2: mass None -> 1

File: tests/data/fixed_floating_joints.urdf (robot description, URDF)
Before this commit: robot fixed_floating_joints, 3 links, 2 joints
Links:
- link Arm_1: mass None -> 1
- link Arm_2: mass None -> 1

File: tests/data/fixed_planar_joints.urdf (robot description, URDF)
Before this commit: robot fixed_planar_joints, 10 links, 8 joints
Links:
- link link1: mass None -> 1
- link planar_negative_x: mass None -> 1
- link planar_negative_y: mass None -> 1
- link planar_negative_z: mass None -> 1
- link planar_tilt: mass None -> 1
- link planar_x: mass None -> 1
- link planar_y: mass None -> 1
- link planar_z: mass None -> 1

File: tests/data/link_skip_ghost_link_with_mimic.urdf (robot description, URDF)
Before this commit: robot link_skip_ghost_link_with_mimic, 4 links, 3 joints
Links:
- link BaseLinkB: mass None -> 1
- link linkB: mass None -> 1

File: tests/data/mimic_joint.urdf (robot description, URDF)
Before this commit: robot mimic_joint, 6 links, 5 joints
Links:
- link BaseLinkB: mass None -> 1
- link linkA: mass None -> 1
- link linkB: mass None -> 1
- link linkC: mass None -> 1
- link linkD: mass None -> 1

File: tests/data/prismatic_joints.urdf (robot description, URDF)
Before this commit: robot prismatic_joints, 6 links, 4 joints
Links:
- link Arm_1: mass None -> 1
- link Arm_2: mass None -> 1
- link Arm_3: mass None -> 1
- link Arm_4: mass None -> 1

File: tests/data/revolute_joints.urdf (robot description, URDF)
Before this commit: robot revolute_joints, 5 links, 4 joints
Links:
- link Arm_1: mass None -> 1
- link Arm_2: mass None -> 1
- link Arm_3: mass None -> 1
- link Arm_4: mass None -> 1

File: tests/data/test_displayname.urdf (robot description, URDF)
Before this commit: robot test_displayname, 5 links, 4 joints
Links:
- link link-box2: mass None -> 1
- link link-box_two_materials_same_names: mass None -> 1
- link link-mesh_dae: mass None -> 1
- link link-mesh_obj: mass None -> 1

File: tests/data/undefined.urdf (robot description, URDF)
Before this commit: robot undefined, 2 links, 1 joints
Links:
- link link_box2: mass None -> 1
